Commit message: Added adaptations for the urdf

File: talos_description/urdf/arm/arm.urdf.xacro (robot description, xacro)
@@ -33,5 +33,5 @@
         <origin xyz="0 0 0" rpy="0 0 0" />
         <geometry>
-          <mesh filename="package://talos_description/meshes/arm/arm_1.STL" scale="1 ${reflect} 1"/>
+          <mesh filename="package://talos_description/meshes/arm/arm_1.dae" scale="1 ${reflect} 1"/>
         </geometry>
         <material name="DarkGrey" />
@@ -62,5 +62,5 @@
         <origin xyz="0 0 0" rpy="0 0 0" />
         <geometry>
-          <mesh filename="package://talos_description/meshes/arm/arm_2.STL" scale="1 ${reflect} 1"/>
+          <mesh filename="package://talos_description/meshes/arm/arm_2.dae" scale="1 ${reflect} 1"/>
         </geometry>
         <material name="DarkGrey" />
@@ -91,5 +91,5 @@
         <origin xyz="0 0 0" rpy="0 0 0" />
         <geometry>
-          <mesh filename="package://talos_description/meshes/arm/arm_3.STL" scale="1 ${reflect} 1"/>
+          <mesh filename="package://talos_description/meshes/arm/arm_3.dae" scale="1 ${reflect} 1"/>
         </geometry>
         <material name="DarkGrey" />
@@ -123,5 +123,5 @@
         <origin xyz="0 0 0" rpy="0 0 0" />
         <geometry>
-          <mesh filename="package://talos_description/meshes/arm/arm_4.STL" scale="1 ${reflect} 1"/>
+          <mesh filename="package://talos_description/meshes/arm/arm_4.dae" scale="1 ${reflect} 1"/>
         </geometry>
         <material name="DarkGrey" />
@@ -150,20 +150,28 @@
      <mu1>0.9</mu1>
      <mu2>0.9</mu2>
+     <!--
      <material>Gazebo/FlatBlack</material>
+     -->
    </gazebo>
    <gazebo reference="${name}_${side}_2_link">
      <mu1>0.9</mu1>
      <mu2>0.9</mu2>
+     <!--
      <material>Gazebo/FlatBlack</material>
+     -->
    </gazebo>
    <gazebo reference="${name}_${side}_3_link">
      <mu1>0.9</mu1>
      <mu2>0.9</mu2>
+     <!--
      <material>Gazebo/FlatBlack</material>
+     -->
    </gazebo>
    <gazebo reference="${name}_${side}_4_link">
      <mu1>0.9</mu1>
      <mu2>0.9</mu2>
+     <!--
      <material>Gazebo/FlatBlack</material>
+     -->
    </gazebo>
    <gazebo reference="${name}_${side}_1_joint">

File: talos_description/urdf/head/head.urdf.xacro (robot description, xacro)
@@ -27,5 +27,5 @@
         <origin xyz="0 0 0" rpy="0 0 0" />
         <geometry>
-          <mesh filename="package://talos_description/meshes/head/head_1.stl" scale="1 1 1"/>
+          <mesh filename="package://talos_description/meshes/head/head_1.dae" scale="1 1 1"/>
         </geometry>
         <material name="DarkGrey" />
@@ -71,5 +71,5 @@
         <origin xyz="0 0 0" rpy="0 0 0" />
         <geometry>
-          <mesh filename="package://talos_description/meshes/head/head_2.stl" scale="1 1 1"/>
+          <mesh filename="package://talos_description/meshes/head/head_2.dae" scale="1 1 1"/>
         </geometry>
         <material name="LightGrey" />

File: talos_description/urdf/torso/torso.urdf.xacro (robot description, xacro)
@@ -25,5 +25,5 @@
         <origin xyz="0 0 0" rpy="0 0 0" />
         <geometry>
-          <mesh filename="package://talos_description/meshes/torso/torso_2.STL" scale="1 1 1"/>
+          <mesh filename="package://talos_description/meshes/torso/torso_2.dae" scale="1 1 1"/>
         </geometry>
         <material name="LightGrey" />
@@ -44,5 +44,5 @@
         <origin xyz="0 0 0" rpy="0 0 0" />
         <geometry>
-          <mesh filename="package://talos_description/meshes/torso/torso_1.STL" scale="1 1 1"/>
+          <mesh filename="package://talos_description/meshes/torso/torso_1.dae" scale="1 1 1"/>
         </geometry>
         <material name="LightGrey" />
@@ -78,5 +78,5 @@
         <origin xyz="0 0 0" rpy="0 0 0" />
         <geometry>
-          <mesh filename="package://talos_description/meshes/torso/base_link.STL" scale="1 1 1"/>
+          <mesh filename="package://talos_description/meshes/torso/base_link.dae" scale="1 1 1"/>
         </geometry>
         <material name="LightGrey" />

Commit message: Added corrected reflected legs

File: talos_description/urdf/arm/arm.urdf.xacro (robot description, xacro)
@@ -33,7 +33,11 @@
         <origin xyz="0 0 0" rpy="0 0 0" />
         <geometry>
-          <mesh filename="package://talos_description/meshes/arm/arm_1.dae" scale="1 ${reflect} 1"/>
-        </geometry>
-        <material name="DarkGrey" />
+          <xacro:if value="${reflect == 1}">
+            <mesh filename="package://talos_description/meshes/arm/arm_1.dae" scale="1 1 1"/>
+          </xacro:if>
+          <xacro:if value="${reflect == -1}">
+            <mesh filename="package://talos_description/meshes/arm/arm_1_reflect1.dae" scale="1 1 1"/>
+          </xacro:if>
+        </geometry>
       </visual>
       <collision>
@@ -62,7 +66,11 @@
         <origin xyz="0 0 0" rpy="0 0 0" />
         <geometry>
-          <mesh filename="package://talos_description/meshes/arm/arm_2.dae" scale="1 ${reflect} 1"/>
-        </geometry>
-        <material name="DarkGrey" />
+          <xacro:if value="${reflect == 1}">
+            <mesh filename="package://talos_description/meshes/arm/arm_2.dae" scale="1 1 1"/>
+          </xacro:if>
+          <xacro:if value="${reflect == -1}">
+            <mesh filename="package://talos_description/meshes/arm/arm_2_reflect.dae" scale="1 1 1"/>
+          </xacro:if>
+        </geometry>
       </visual>
       <collision>
@@ -91,7 +99,11 @@
         <origin xyz="0 0 0" rpy="0 0 0" />
         <geometry>
-          <mesh filename="package://talos_description/meshes/arm/arm_3.dae" scale="1 ${reflect} 1"/>
-        </geometry>
-        <material name="DarkGrey" />
+          <xacro:if value="${reflect == 1}">
+            <mesh filename="package://talos_description/meshes/arm/arm_3.dae" scale="1 1 1"/>
+          </xacro:if>
+          <xacro:if value="${reflect == -1}">
+            <mesh filename="package://talos_description/meshes/arm/arm_3_reflect.dae" scale="1 1 1"/>
+          </xacro:if>
+        </geometry>
       </visual>
       <collision>
@@ -123,7 +135,11 @@
         <origin xyz="0 0 0" rpy="0 0 0" />
         <geometry>
-          <mesh filename="package://talos_description/meshes/arm/arm_4.dae" scale="1 ${reflect} 1"/>
-        </geometry>
-        <material name="DarkGrey" />
+          <xacro:if value="${reflect == 1}">
+            <mesh filename="package://talos_description/meshes/arm/arm_4.dae" scale="1 1 1"/>
+          </xacro:if>
+          <xacro:if value="${reflect == -1}">
+            <mesh filename="package://talos_description/meshes/arm/arm_4_reflect.dae" scale="1 1 1"/>
+          </xacro:if>
+        </geometry>
       </visual>
       <collision>
@@ -150,28 +166,16 @@
      <mu1>0.9</mu1>
      <mu2>0.9</mu2>
-     <!--
-     <material>Gazebo/FlatBlack</material>
-     -->
    </gazebo>
    <gazebo reference="${name}_${side}_2_link">
      <mu1>0.9</mu1>
      <mu2>0.9</mu2>
-     <!--
-     <material>Gazebo/FlatBlack</material>
-     -->
    </gazebo>
    <gazebo reference="${name}_${side}_3_link">
      <mu1>0.9</mu1>
      <mu2>0.9</mu2>
-     <!--
-     <material>Gazebo/FlatBlack</material>
-     -->
    </gazebo>
    <gazebo reference="${name}_${side}_4_link">
      <mu1>0.9</mu1>
      <mu2>0.9</mu2>
-     <!--
-     <material>Gazebo/FlatBlack</material>
-     -->
    </gazebo>
    <gazebo reference="${name}_${side}_1_joint">

File: talos_description/urdf/gripper/gripper.urdf.xacro (robot description, xacro)
@@ -11,5 +11,5 @@
                 <origin xyz="0 0 0" rpy="0 0 0" />
                 <geometry>
-                  <mesh filename="package://talos_description/meshes/gripper/base_link.STL" scale="1 1 1"/>
+                  <mesh filename="package://talos_description/meshes/gripper/base_link.dae" scale="1 1 1"/>
                 </geometry>
                 <material name="DarkGrey"/>
@@ -34,5 +34,5 @@
                 <origin xyz="0 0 0" rpy="0 0 0" />
                 <geometry>
-                  <mesh filename="package://talos_description/meshes/gripper/gripper_motor_double.STL" scale="1 1 1"/>
+                  <mesh filename="package://talos_description/meshes/gripper/gripper_motor_double.dae" scale="1 1 1"/>
                 </geometry>
               <material name="Orange"/>
@@ -59,5 +59,5 @@
                 <origin xyz="0 0 0" rpy="0 0 0" />
                 <geometry>
-                  <mesh filename="package://talos_description/meshes/gripper/inner_double.STL" scale="1 1 1"/>
+                  <mesh filename="package://talos_description/meshes/gripper/inner_double.dae" scale="1 1 1"/>
                 </geometry>
               <material name="Orange"/>
@@ -84,5 +84,5 @@
                 <origin xyz="0 0 0" rpy="0 0 0" />
                 <geometry>
-                  <mesh filename="package://talos_description/meshes/gripper/fingertip.STL" scale="1 1 1"/>
+                  <mesh filename="package://talos_description/meshes/gripper/fingertip.dae" scale="1 1 1"/>
                 </geometry>
               <material name="DarkGrey"/>
@@ -109,5 +109,5 @@
                 <origin xyz="0 0 0" rpy="0 0 0" />
                 <geometry>
-                  <mesh filename="package://talos_description/meshes/gripper/fingertip.STL" scale="1 1 1"/>
+                  <mesh filename="package://talos_description/meshes/gripper/fingertip.dae" scale="1 1 1"/>
                 </geometry>
                 <material name="DarkGrey"/>
@@ -134,5 +134,5 @@
                 <origin xyz="0 0 0" rpy="0 0 0" />
                 <geometry>
-                  <mesh filename="package://talos_description/meshes/gripper/gripper_motor_single.STL" scale="1 1 1"/>
+                  <mesh filename="package://talos_description/meshes/gripper/gripper_motor_single.dae" scale="1 1 1"/>
                 </geometry>
               <material name="Orange"/>
@@ -159,5 +159,5 @@
                 <origin xyz="0 0 0" rpy="0 0 0" />
                 <geometry>
-                  <mesh filename="package://talos_description/meshes/gripper/inner_single.STL" scale="1 1 1"/>
+                  <mesh filename="package://talos_description/meshes/gripper/inner_single.dae" scale="1 1 1"/>
                 </geometry>
               <material name="Orange"/>
@@ -184,5 +184,5 @@
                 <origin xyz="0 0 0" rpy="0 0 0" />
                 <geometry>
-                  <mesh filename="package://talos_description/meshes/gripper/fingertip.STL" scale="1 1 1"/>
+                  <mesh filename="package://talos_description/meshes/gripper/fingertip.dae" scale="1 1 1"/>
                 </geometry>
               <material name="DarkGrey"/>
@@ -206,11 +206,4 @@
         <xacro:virtual_joints name="${name}" />
         <xacro:gripper_transmission name="${name}" reduction="1.0" />
-        <!-- virtual mimic joints -->
-<!--         <xacro:gripper_virtual_transmission name="${name}_inner_double" reduction="1.0"/>
-        <xacro:gripper_virtual_transmission name="${name}_fingertip_1" reduction="1.0"/>
-        <xacro:gripper_virtual_transmission name="${name}_fingertip_2" reduction="1.0"/>
-        <xacro:gripper_virtual_transmission name="${name}_inner_single" reduction="1.0"/>
-        <xacro:gripper_virtual_transmission name="${name}_motor_single" reduction="1.0"/>
-        <xacro:gripper_virtual_transmission name="${name}_fingertip_3" reduction="1.0"/> -->
   </xacro:macro>
 </robot>

File: talos_description/urdf/leg/leg.urdf.xacro (robot description, xacro)
@@ -15,7 +15,11 @@
         <origin rpy="0 0 0" xyz="0 0 0"/>
         <geometry>
-          <mesh filename="package://talos_description/meshes/v2/hip_z_lo_res.stl" scale="1 ${reflect*1} 1"/>
-        </geometry>
-        <material name="DarkGrey" />
+          <xacro:if value="${reflect == 1}">
+            <mesh filename="package://talos_description/meshes/v2/hip_z_lo_res.dae" scale="1 1 1"/>
+          </xacro:if>
+          <xacro:if value="${reflect == -1}">
+            <mesh filename="package://talos_description/meshes/v2/hip_z_lo_res_reflect.dae" scale="1 1 1"/>
+          </xacro:if>
+        </geometry>
       </visual>
       <collision>
@@ -41,7 +45,11 @@
         <origin xyz="0 0 0.0" rpy="0  0  0" />
         <geometry>
-          <mesh filename="package://talos_description/meshes/v2/hip_x_lo_res.stl" scale="1 ${reflect*1} 1"/>
-        </geometry>
-        <material name="DarkGrey" />
+          <xacro:if value="${reflect == 1}">
+            <mesh filename="package://talos_description/meshes/v2/hip_x_lo_res.dae" scale="1 1 1"/>
+          </xacro:if>
+          <xacro:if value="${reflect == -1}">
+            <mesh filename="package://talos_description/meshes/v2/hip_x_lo_res_reflect.dae" scale="1 1 1"/>
+          </xacro:if>
+        </geometry>
       </visual>
       <collision>
@@ -67,7 +75,11 @@
         <origin rpy="0 0 0" xyz="0 0 0"/>
         <geometry>
-          <mesh filename="package://talos_description/meshes/v2/hip_y_lo_res.stl" scale="1 ${reflect*1} 1"/>
-        </geometry>
-        <material name="DarkGrey" />
+          <xacro:if value="${reflect == 1}">
+            <mesh filename="package://talos_description/meshes/v2/hip_y_lo_res.dae" scale="1 1 1"/>
+          </xacro:if>
+          <xacro:if value="${reflect == -1}">
+            <mesh filename="package://talos_description/meshes/v2/hip_y_lo_res_reflect.dae" scale="1 1 1"/>
+          </xacro:if>
+        </geometry>
       </visual>
       <collision>
@@ -93,7 +105,11 @@
         <origin rpy="0 0 0" xyz="0 0 0"/>
         <geometry>
-          <mesh filename="package://talos_description/meshes/v2/knee_lo_res.stl" scale="1 ${reflect*1} 1"/>
-        </geometry>
-        <material name="DarkGrey" />
+          <xacro:if value="${reflect == 1}">
+            <mesh filename="package://talos_description/meshes/v2/knee_lo_res.dae" scale="1 1 1"/>
+          </xacro:if>
+          <xacro:if value="${reflect == -1}">
+            <mesh filename="package://talos_description/meshes/v2/knee_lo_res_reflect.dae" scale="1 1 1"/>
+          </xacro:if>
+        </geometry>
       </visual>
       <collision>
@@ -120,7 +136,11 @@
         <origin xyz="0 0 0.0" rpy="0 0 0" />
         <geometry>
-          <mesh filename="package://talos_description/meshes/v2/ankle_Y_lo_res.stl" scale="1 ${reflect*1} 1"/>
-        </geometry>
-        <material name="Grey" />
+          <xacro:if value="${reflect == 1}">
+            <mesh filename="package://talos_description/meshes/v2/ankle_Y_lo_res.dae" scale="1 1 1"/>
+          </xacro:if>
+          <xacro:if value="${reflect == -1}">
+            <mesh filename="package://talos_description/meshes/v2/ankle_Y_lo_res_reflect.dae" scale="1 1 1"/>
+          </xacro:if>
+        </geometry>
       </visual>
       <collision>
@@ -146,7 +166,11 @@
         <origin rpy="0 0 0" xyz="0 0 0"/>
         <geometry>
-          <mesh filename="package://talos_description/meshes/v2/ankle_X_lo_res.stl" scale="1 ${reflect*1} 1"/>
-        </geometry>
-        <material name="Grey" />
+          <xacro:if value="${reflect == 1}">
+            <mesh filename="package://talos_description/meshes/v2/ankle_X_lo_res.dae" scale="1 1 1"/>
+          </xacro:if>
+          <xacro:if value="${reflect == -1}">
+            <mesh filename="package://talos_description/meshes/v2/ankle_X_lo_res_reflect.dae" scale="1 1 1"/>
+          </xacro:if>
+        </geometry>
       </visual>
       <xacro:talos_foot_collision />
